File: Schematics/z80console.kicad_sch (KiCad schematic)
At the start: 11 parts, among them U1 Z80CPU, U2 AT28C64B-15PU, U3 74HCT02, U4 74HC04, U5 74HCT85, U6 NE555P, U7 74HC04

Commit message: changes
Parts:
- added U11: 74HCT85, symbol 74xx:74HCT85
- added U12: 74HC04, symbol 74xx:74HC04
- added U8: MK6264LN-70, symbol Symbols:MK6264LN-70
- added U9: 74HCT00, symbol 74xx:74HCT00
Connections:
- net +5V: now also U11.11 (B1), U11.14 (B2), U11.16 (VCC), U11.2 (Ia<b), U8.26 (E2), U8.28 (VCC)
- net A12: now also U11.10 (A0)
- net A13: now also U11.12 (A1)
- net A14: now also U11.13 (A2)
- net A15: now also U11.15 (A3)
- net GND: now also U11.1 (B3), U11.3 (Ia=b), U11.4 (Ia>b), U11.8 (GND), U11.9 (B0), U8.14 (VSS), U8.20 (~{E1}), U8.46 (VSS)
- net ROM COMP: now also U5.7 (Oa<b); no longer U5.6 (Oa=b)
- net ~{MREQ}: now also U9.10, U9.9
- net ~{WR}: now also U8.27 (~{W})
- new net: U12.2, U9.1
- new net: U9.12, U9.6
- new net: U9.13, U9.8
- new net: U9.3, U9.4, U9.5
- new net RAM COMP: U11.7 (Oa<b), U9.2
- new net RAM ~{G}: U8.22 (~{G}), U9.11
- new net ROM COMP 2: U12.1
Other:
- note added: "RAM LOGIC"
