File: Schematics - OLD/z80console.kicad_sch (KiCad schematic)
At the start: 15 parts, among them U1 Z80CPU, U11 74HCT85, U12 74HC04, U2 AT28C64B-15PU, U3 74HCT02, U4 74HC04, U5 74HCT85, U6 NE555P, U7 74HC04, U8 MK6264LN-70, U9 74HCT00

Commit message: commit
Parts:
- removed U3: 74HCT02, symbol 74xx:74HCT02
- removed U9: 74HCT00, symbol 74xx:74HCT00
- added U10: 74HCT85, symbol 74xx:74HCT85
- added U3, U9: 74LS32, symbol 74xx:74LS32
Connections:
- net +5V: now also U10.14 (B2), U10.16 (VCC), U10.2 (Ia<b)
- net A12: now also U10.10 (A0)
- net A13: now also U10.12 (A1)
- net A14: now also U10.13 (A2)
- net A15: now also U10.15 (A3)
- net GND: now also U10.1 (B3), U10.11 (B1), U10.3 (Ia=b), U10.4 (Ia>b), U10.8 (GND), U10.9 (B0)
- net RAM COMP: now also U12.1
- net RAM ~{G}: now also U9.6
- net ROM COMP 2: now also U10.7 (Oa<b), U9.1; no longer U12.1
- net ROM ~{OE}: now also U3.6
- net ~{MREQ}: now also U3.2, U9.5
- net ~{RD}: now also U3.1
- net at U12.2: now also U9.2
- net at U4.2: now also U3.5
- new net: U9.3, U9.4
- new net: U3.3, U3.4
Other:
- note added: "(ROM_COMP_2 + ~{RAM_COMP}) + ~{MREQ}"
- note added: "ROM (2) LOGIC"
- moved on the sheet: U12A, U4A
